Commit message: add move rviz, but it's not correct

File: turtle_brick/urdf/my_robot.urdf (robot description, URDF)
Before this commit: robot my_robot, 6 links, 5 joints
Links:
- removed link lidar
Joints:
- removed joint base_lidar_joint

Commit message: frames loading properly

File: turtle_brick/urdf/my_robot.urdf (robot description, URDF)
Before this commit: robot my_robot, 5 links, 4 joints
Links:
- removed link left_wheel
- removed link right_wheel
Joints:
- removed joint base_left_wheel_joint
- removed joint base_right_wheel_joint

Commit message: add correct shapes

File: turtle_brick/urdf/my_robot.urdf (robot description, URDF)
Before this commit: robot my_robot, 3 links, 2 joints
Links:
- added link pole_link; visual cylinder length=0.4 radius=0.025
- added link top_link; visual cylinder length=0.05 radius=0.3
- link base_link: geometry visual box size=0.2 0.2 0.2
- link caster_wheel: geometry visual cylinder length=0.05 radius=0.1
Joints:
- added joint pole_to_base_joint: type fixed, parent base_link, child pole_link, origin xyz=0 0 0.4 rpy=0 0 0
- added joint top_wheel_joint: type continuous, parent pole_link, child top_link, origin xyz=0.0 0 0.2 rpy=0 0 0
- joint base_caster_wheel_joint: origin xyz=0.2 0 -0.05 rpy=0 0 0 -> xyz=0.2 0 0.1055 rpy=0 0 0
