Commit message: fix joint continuous joint type publish error

File: turtle_brick/urdf/turtle.urdf.xacro (robot description, xacro)
@@ -39,20 +39,4 @@
         <origin xyz="0 0 0.4" rpy="0 0 0"/>
     </joint>
-    <!-- Caster wheel link -->
-    <link name="caster_wheel">
-        <visual>
-            <geometry>
-                 <cylinder radius="0.1" length="0.05"/>
-            </geometry>
-             <origin xyz="0.0 0.0 -0.0" rpy="1.57 0.0 0.0"/>
-        </visual>
-    </link>
-    <!-- Caster wheel joint -->
-    <joint name="base_caster_wheel_joint" type="continuous">
-        <parent link="base_link"/>
-        <child link="caster_wheel"/>
-        <origin xyz="0.2 0 0.1055" rpy="0 0 0"/>
-        <axis xyz="0.0 1.0 0.0"/>
-    </joint>
     <link name="top_link">
         <visual>
@@ -64,5 +48,5 @@
         </visual>
     </link>
-    <joint name="top_wheel_joint" type="continuous">
+    <joint name="top_wheel_joint" type="fixed">
         <parent link="pole_link"/>
         <child link="top_link"/>
@@ -77,3 +61,19 @@
         <origin xyz="0.0 0 0.1" rpy="0 0 0"/>
     </joint>
+    <!-- Caster wheel link -->
+    <link name="caster_wheel">
+        <visual>
+            <geometry>
+                 <cylinder radius="0.1" length="0.05"/>
+            </geometry>
+             <origin xyz="0.0 0.0 0.0" rpy="1.57 0.0 0.0"/>
+        </visual>
+    </link>
+    <!-- Caster wheel joint -->
+    <joint name="caster_wheel_joint" type="continuous">
+        <parent link="base_link"/>
+        <child link="caster_wheel"/>
+        <origin xyz="0.0 0.0 0.0" rpy="0 0 0"/>
+        <axis xyz="0.0 1.0 0.0"/>
+    </joint>
 </robot>

Commit message: add holonomic

File: turtle_brick/urdf/turtle.urdf.xacro (robot description, xacro)
@@ -4,5 +4,5 @@
 <xacro:property name="body" value="0.6" />
     <material name="grey">
-        <color rgba="0.7 0.7 0.7 1"/>
+        <color rgba="0.7 0.7 0.7 1.0"/>
     </material>
     <material name="green">
@@ -10,8 +10,8 @@
     </material>
     <material name="white">
-        <color rgba="1 1 1 1"/>
+        <color rgba="1.0 1.0 1.0 1.0"/>
     </material>
     <material name="blue">
-        <color rgba="0.15 0.2 0.4 1"/>
+        <color rgba="0.15 0.2 0.4 1.0"/>
     </material>
     <!-- Base of the robot -->
@@ -21,5 +21,5 @@
                 <box size="0.2 0.2 0.2"/>
             </geometry>
-            <origin xyz="0 0 0.20" rpy="0 0 0"/>
+            <origin xyz="0.0 0.0 0.20" rpy="0.0 0.0 0.0"/>
             <material name="green"/>
         </visual>
@@ -30,5 +30,5 @@
                     <cylinder radius="0.025" length="0.4"/>
             </geometry>
-            <origin xyz="0 0 0" rpy="0 0 0"/>
+            <origin xyz="0.0 0.0 0.4" rpy="0.0 0.0 0.0"/>
             <material name="grey"/>
         </visual>
@@ -37,5 +37,5 @@
         <parent link="base_link"/>
         <child link="pole_link"/>
-        <origin xyz="0 0 0.4" rpy="0 0 0"/>
+        <origin xyz="0.0 0.0 0.0" rpy="0.0 0.0 0.0"/>
     </joint>
     <link name="top_link">
@@ -44,5 +44,5 @@
                  <cylinder radius="0.3" length="0.05"/>
             </geometry>
-             <origin xyz="0.0 0.0 -0.0" rpy="0 0.0 0.0"/>
+             <origin xyz="0.0 0.0 0.6" rpy="0.0 0.0 0.0"/>
              <material name="blue"/>
         </visual>
@@ -51,5 +51,5 @@
         <parent link="pole_link"/>
         <child link="top_link"/>
-        <origin xyz="0.0 0 0.2" rpy="0 0 0"/>
+        <origin xyz="0.0 0.0 0.0" rpy="0.0 0.0 0.0"/>
     </joint>
     <!-- Base footprint link -->
@@ -59,5 +59,5 @@
         <parent link="base_footprint"/>
         <child link="base_link"/>
-        <origin xyz="0.0 0 0.1" rpy="0 0 0"/>
+        <origin xyz="0.0 0.0 0.1" rpy="0.0 0.0 0.0"/>
     </joint>
     <!-- Caster wheel link -->
@@ -74,5 +74,5 @@
         <parent link="base_link"/>
         <child link="caster_wheel"/>
-        <origin xyz="0.0 0.0 0.0" rpy="0 0 0"/>
+        <origin xyz="0.0 0.0 0.0" rpy="0.0 0.0 0.0"/>
         <axis xyz="0.0 1.0 0.0"/>
     </joint>

Commit message: add physics & fix gaps between start and arena requirements

File: turtle_brick/urdf/turtle.urdf.xacro (robot description, xacro)
@@ -39,5 +39,5 @@
         <origin xyz="0.0 0.0 0.0" rpy="0.0 0.0 0.0"/>
     </joint>
-    <link name="top_link">
+    <link name="platform">
         <visual>
             <geometry>
@@ -50,5 +50,5 @@
     <joint name="top_wheel_joint" type="fixed">
         <parent link="pole_link"/>
-        <child link="top_link"/>
+        <child link="platform"/>
         <origin xyz="0.0 0.0 0.0" rpy="0.0 0.0 0.0"/>
     </joint>
@@ -62,5 +62,5 @@
     </joint>
     <!-- Caster wheel link -->
-    <link name="caster_wheel">
+    <link name="wheel">
         <visual>
             <geometry>
@@ -71,7 +71,7 @@
     </link>
     <!-- Caster wheel joint -->
-    <joint name="caster_wheel_joint" type="continuous">
+    <joint name="wheel_joint" type="continuous">
         <parent link="base_link"/>
-        <child link="caster_wheel"/>
+        <child link="wheel"/>
         <origin xyz="0.0 0.0 0.0" rpy="0.0 0.0 0.0"/>
         <axis xyz="0.0 1.0 0.0"/>

Commit message: fix turtle_node

File: turtle_brick/urdf/turtle.urdf.xacro (robot description, xacro)
@@ -1,6 +1,8 @@
 <?xml version="1.0"?>
 <robot name="my_robot" xmlns:xacro="http://www.ros.org/wiki/xacro" >
-<xacro:property name="platform height" value="0.2" />
-<xacro:property name="body" value="0.6" />
+    <xacro:arg name="platform_height" default="0.2"/>
+    <xacro:arg name="wheel_radius" default="0.1"/>
+    <xacro:property name="platform_height" value="$(arg platform_height)" />
+    <xacro:property name="wheel_radius" value="$(arg wheel_radius)" />
     <material name="grey">
         <color rgba="0.7 0.7 0.7 1.0"/>
@@ -44,5 +46,5 @@
                  <cylinder radius="0.3" length="0.05"/>
             </geometry>
-             <origin xyz="0.0 0.0 0.6" rpy="0.0 0.0 0.0"/>
+             <origin xyz="0.0 0.0 $(arg platform_height)" rpy="0.0 0.0 0.0"/>
              <material name="blue"/>
         </visual>
@@ -65,5 +67,5 @@
         <visual>
             <geometry>
-                 <cylinder radius="0.1" length="0.05"/>
+                 <cylinder radius="$(arg wheel_radius)" length="0.05"/>
             </geometry>
              <origin xyz="0.0 0.0 0.0" rpy="1.57 0.0 0.0"/>

Commit message: add caught the brick

File: turtle_brick/urdf/turtle.urdf.xacro (robot description, xacro)
@@ -5,4 +5,5 @@
     <xacro:property name="platform_height" value="$(arg platform_height)" />
     <xacro:property name="wheel_radius" value="$(arg wheel_radius)" />
+        <xacro:property name="platform_radius" value="$(arg platform_radius)" />
     <material name="grey">
         <color rgba="0.7 0.7 0.7 1.0"/>
@@ -44,5 +45,5 @@
         <visual>
             <geometry>
-                 <cylinder radius="0.3" length="0.05"/>
+                 <cylinder radius="$(arg platform_radius)" length="0.05"/>
             </geometry>
              <origin xyz="0.0 0.0 $(arg platform_height)" rpy="0.0 0.0 0.0"/>

Commit message: fix wheel rotation state

File: turtle_brick/urdf/turtle.urdf.xacro (robot description, xacro)
@@ -51,8 +51,10 @@
         </visual>
     </link>
-    <joint name="top_wheel_joint" type="fixed">
+    <joint name="top_wheel_joint" type="revolute">
         <parent link="pole_link"/>
         <child link="platform"/>
         <origin xyz="0.0 0.0 0.0" rpy="0.0 0.0 0.0"/>
+        <axis xyz="1.0 0.0 0.0"/>
+        <limit lower="-0.5" upper="0.5" effort="5.0" velocity="1.0"/>
     </joint>
     <!-- Base footprint link -->
@@ -74,9 +76,10 @@
     </link>
     <!-- Caster wheel joint -->
-    <joint name="wheel_joint" type="continuous">
+    <joint name="wheel_joint" type="revolute">
         <parent link="base_link"/>
         <child link="wheel"/>
         <origin xyz="0.0 0.0 0.0" rpy="0.0 0.0 0.0"/>
         <axis xyz="0.0 1.0 0.0"/>
+        <limit lower="-3.1" upper="3.1" effort="5.0" velocity="1.0"/>
     </joint>
 </robot>

Commit message: fix platform joint

File: turtle_brick/urdf/turtle.urdf.xacro (robot description, xacro)
@@ -51,10 +51,10 @@
         </visual>
     </link>
-    <joint name="top_wheel_joint" type="revolute">
+    <joint name="platform_joint" type="revolute">
         <parent link="pole_link"/>
         <child link="platform"/>
         <origin xyz="0.0 0.0 0.0" rpy="0.0 0.0 0.0"/>
         <axis xyz="1.0 0.0 0.0"/>
-        <limit lower="-0.5" upper="0.5" effort="5.0" velocity="1.0"/>
+        <limit lower="-0.5" upper="0.5" effort="1.0" velocity="1.0"/>
     </joint>
     <!-- Base footprint link -->
